File: 3. Design/7. PCB/stm32f0-qfp32-devboard/stm32f0-qfp32-devboard.brd (EAGLE design)
At the start: 18.3 x 34.6 mm, 12 parts, among them IC1 STM32F051

Commit message: ADD|UPDT|FIX: Corrected Dev Board exports and finished wristband board's schematic
Parts:
- removed FRAME2: FRAME-LETTERNO_PACKAGE, SparkFun-Aesthetics:DUMMY
Changed lines of the file:
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@@
 <drawing>
 <settings>
-<setting alwaysvectorfont="yes"/>
+<setting alwaysvectorfont="no"/>
 <setting keepoldvectorfont="yes"/>
 <setting verticaltext="up"/>
@@
 <attribute name="VALUE" x="3.8354" y="30.2514" size="0.6096" layer="27" font="vector" ratio="20"/>
 </element>
-<element name="FRAME2" library="SparkFun-Aesthetics" library_urn="urn:adsk.eagle:library:507" package="DUMMY" package3d_urn="urn:adsk.eagle:package:37104/1" value="FRAME-LETTERNO_PACKAGE" x="-1.016" y="-0.635" smashed="yes">
-<attribute name="DESIGNER" value="Nobody" x="-1.016" y="-0.635" size="1.778" layer="27" display="off"/>
-<attribute name="VERSION" value="v01" x="-1.016" y="-0.635" size="1.778" layer="27" display="off"/>
-</element>
 </elements>
