File: 3. Design/7. PCB/wristband/wristband-pcb.brd (EAGLE design)
At the start: 27.5 x 36.3 mm, 44 parts, among them IC1 STM32F051K8T6, Y2 FA-20H_16.0000MF12Z-AC3, Y3 FA-20H_16.0000MF12Z-AC3

Commit message: UPDT: Functional part of the wristband PCB done
Parts:
- moved C8 0.51 mm to (14.0, 27.7), turned to 0 degrees
Routing:
- net VDD: track 86.6 -> 94.0 mm, vias 3 -> 4
- net VCC_BATT: track 16.9 -> 17.4 mm
- net GND: track 0.00 -> 0.15 mm, vias 4 -> 3
